File: KiCad files/karve-split.kicad_pcb (KiCad board)
At the start: 2 copper layers, 352.7 x 140.2 mm, 221 parts, among them J2 USB_C_Receptacle_USB2.0_16P, J3 USB_C_Receptacle_USB2.0_16P, SW100 SW_Push, SW101 SW_Push, SW102 SW_Push, SW103 SW_Push, SW104 SW_Push, SW105 SW_Push, SW106 SW_Push, SW107 SW_Push, SW108 SW_Push, SW109 SW_Push, SW110 SW_Push, SW111 SW_Push, SW112 SW_Push, SW113 SW_Push, SW114 SW_Push, SW115 SW_Push, SW116 SW_Push, SW117 SW_Push, SW118 SW_Push, SW119 SW_Push, SW120 SW_Push, SW121 SW_Push, SW122 SW_Push, SW123 SW_Push, SW124 SW_Push, SW125 SW_Push, SW126 SW_Push, SW127 SW_Push, SW128 SW_Push, SW129 SW_Push, SW130 SW_Push, SW131 SW_Push, SW132 SW_Push, SW133 SW_Push, SW134 SW_Push, SW43 SW_Push, SW44 SW_Push, SW45 SW_Push, SW46 SW_Push, SW47 SW_Push, SW48 SW_Push, SW49 SW_Push, SW50 SW_Push, SW51 RotaryEncoder_Switch, SW52 SW_Push, SW53 SW_Push, SW54 SW_Push, SW55 SW_Push, SW56 SW_Push, SW57 SW_Push, SW58 SW_Push, SW59 SW_Push, SW60 SW_Push, SW61 SW_Push, SW62 SW_Push, SW63 SW_Push, SW64 SW_Push, SW65 SW_Push, SW66 SW_Push, SW67 SW_Push, SW68 SW_Push, SW69 SW_Push, SW70 SW_Push, SW71 SW_Push, SW72 SW_Push, SW73 SW_Push, SW74 SW_Push, SW75 SW_Push, SW76 SW_Push, SW77 SW_Push, SW78 SW_Push, SW79 SW_Push, SW80 SW_Push, SW81 SW_Push, SW82 SW_Push, SW83 SW_Push, SW84 SW_Push, SW85 SW_Push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

Commit message: update readme and all kicad-related files
Parts:
- moved D48 3.58 mm to (137.7, 72.0)
- moved D97 1.00 mm to (295.2, 68.8)
Routing:
- net Net-(D97-A): track 3.83 -> 0.00 mm
- net /Right Split/ROW0: track 209.7 -> 211.5 mm
- net /Right Split/COL4: track 180.2 -> 179.1 mm
- net /Left Split/ROW0: track 122.2 -> 122.8 mm
- net /Right Split/COL6: track 206.1 -> 206.5 mm, vias 0 -> 2

Commit message: updated gerber and kicad files, as well as added journal.md file
Parts:
- added G***: LOGO, LOGO, F.Cu at (359.7, 117.8)
- added G***: LOGO, LOGO, F.Cu at (31.0, 119.5)
Routing:
- net Net-(D97-A): track 0.00 -> 3.46 mm
